File: kicad/extruder.kicad_pcb (KiCad board)
At the start: 2 copper layers, 51.7 x 53.7 mm, 29 parts, among them P1 therm, P10 winder, P11 enc, P12 icsp, P13 pwr, P14 24V, P15 5V, P2 lcd, P3 buzzer, P4 qc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

Commit message: updated schematic
Parts:
- removed REF** (x4): 1pin, Connect:1pin
- added D1: D, Diodes_SMD:DO-214AC, F.Cu at (137.3, 50.3)
- added D2: D, Diodes_SMD:DO-214AC, F.Cu at (144.1, 53.1)
- added D3: D, Diodes_SMD:DO-214AC, F.Cu at (155.1, 50.3)
- added R1: R100k, Resistors_SMD:R_0603, F.Cu at (135.1, 69.7)
- added R2: R100k, Resistors_SMD:R_0603, F.Cu at (142.7, 69.7)
- added R3: R100k, Resistors_SMD:R_0603, F.Cu at (154.1, 68.4)
- added REF**111: 1pin, Connect:1pin, F.Cu at (119.9, 46.1)
- added REF**112: 1pin, Connect:1pin, F.Cu at (119.9, 96.1)
- added REF**121: 1pin, Connect:1pin, F.Cu at (163.9, 46.1)
- added REF**122: 1pin, Connect:1pin, F.Cu at (163.9, 96.1)
- C1, C2: footprint Capacitors_SMD:C_0603 -> Capacitors_SMD:C_0805
- P10: value winder -> auger; footprint Pin_Headers:Pin_Header_Straight_1x02 -> screw_terminals:2Screw
- P9: value auger -> winder; footprint screw_terminals:2Screw -> Pin_Headers:Pin_Header_Straight_1x02
- PSU1: footprint 7-28V -> DC-DC_Buck:7-28V
- Q1: value qhtr -> IRLR2905PBF
- Q2: value qauger -> IRLR2905PBF
- Q3: value qwinder -> IRLR2905PBF
- moved P12 1.40 mm to (118.6, 66.5)
- moved P6 1.27 mm to (118.6, 60.5)
Connections:
- P5 pad 4: txd -> rxd
- P5 pad 5: rxd -> txd
- Q2 pad 1: auger -> winder
- Q3 pad 1: winder -> auger
- cpu1 pad 10: auger -> winder
- cpu1 pad 12: (no net) -> auger
- cpu1 pad 13: winder -> servo
- cpu1 pad 14: servo -> (no net)
Routing:
- net GND: track 354.2 -> 288.8 mm
- net auger: track 24.2 -> 38.1 mm
- net +24V: track 54.1 -> 64.4 mm
- net winder: track 35.5 -> 26.8 mm
- net rxd: track 28.4 -> 34.8 mm
- net Net-(D3-Pad2): track 6.01 -> 10.7 mm
- net Net-(D1-Pad2): track 7.14 -> 11.4 mm
- net htr: track 11.8 -> 14.5 mm
- net Net-(D2-Pad2): track 7.88 -> 10.2 mm
- net VCC: track 154.6 -> 156.0 mm
- net txd: track 27.6 -> 26.4 mm
- net servo: track 22.7 -> 23.7 mm
- net miso: track 13.1 -> 13.6 mm
- net sck: track 14.1 -> 14.7 mm
Other:
- board size 51.7 x 53.7 mm -> 51.7 x 59.4 mm

Commit message: updated electronics
Parts:
- removed REF**111, REF**112, REF**121, REF**122: 1pin, Connect:1pin
- added P16: CONN_01X01, Connect:1pin, F.Cu at (163.9, 96.1)
- added P17: CONN_01X01, Connect:1pin, F.Cu at (115.0, 46.0)
- added P18: CONN_01X01, Connect:1pin, F.Cu at (164.0, 46.0)
- added W1: TEST_1P, Pin_Headers:Pin_Header_Straight_1x01, B.Cu at (117.3, 81.1)
- added W3: TEST_1P, Pin_Headers:Pin_Header_Straight_1x01, B.Cu at (134.2, 91.7)
- added W4: TEST_1P, Pin_Headers:Pin_Header_Straight_1x01, B.Cu at (135.0, 73.3)
- C1, C2: value C22uF -> C22pF
- P3: value buzzer -> CONN_01X01; footprint Pin_Headers:Pin_Header_Straight_1x02 -> Connect:1pin; moved to F.Cu
- moved P3 42.8 mm to (115.0, 96.1), turned to 0 degrees
Connections:
- P3 pad 1: bzr -> (no net)
- P4 pad 3: length -> diam
- P4 pad 4: diam -> length
- cpu1 pad 11: (no net) -> Net-(W4-Pad1)
- cpu1 pad 19: (no net) -> Net-(W1-Pad1)
- cpu1 pad 22: length -> diam
- cpu1 pad 23: diam -> length
- cpu1 pad 26: bzr -> Net-(W3-Pad1)
Routing:
- net bzr: track 35.6 -> 0.00 mm
- net Net-(W1-Pad1): track 0.00 -> 15.2 mm
- net Net-(W3-Pad1): track 0.00 -> 6.01 mm
- net Net-(W4-Pad1): track 0.00 -> 4.88 mm
- net VCC: track 156.0 -> 159.2 mm
- net GND: track 288.8 -> 291.8 mm
- net htr: track 14.5 -> 15.8 mm
- net winder: track 26.8 -> 27.9 mm
- net rxd: track 34.8 -> 35.6 mm
- net sda: track 26.6 -> 26.1 mm
- net mosi: track 18.6 -> 19.2 mm
- added copper zone on F.Cu, net Net-(W1-Pad1)
- added copper zone on F.Cu, net Net-(W3-Pad1)
- added copper zone on F.Cu, net Net-(W4-Pad1)
Other:
- board size 51.7 x 59.4 mm -> 56.8 x 59.4 mm
