File: kicad/extruder.sch (KiCad schematic (older format))
At the start: 25 parts, among them P1 therm, P10 winder, P11 enc, P12 icsp, P13 pwr, P14 24V, P15 5V, P2 lcd, P3 buzzer, P4 qc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

Commit message: updated schematic
Parts:
- added D1, D2, D3: D, Diodes_SMD:DO-214AC, symbol D
- added R1, R2, R3: R100k, Resistors_SMD:R_0603, symbol R
- C1, C2: footprint Capacitors_SMD:C_0603 -> Capacitors_SMD:C_0805
- P10: value winder -> auger; footprint Pin_Headers:Pin_Header_Straight_1x02 -> screw_terminals:2Screw
- P9: value auger -> winder; footprint screw_terminals:2Screw -> Pin_Headers:Pin_Header_Straight_1x02
- Q1: value qhtr -> IRLR2905PBF
- Q2: value qauger -> IRLR2905PBF
- Q3: value qwinder -> IRLR2905PBF
Connections:
- wire segments 40 -> 55
Other:
- moved on the sheet: P10, P8, P9

Commit message: updated electronics
Parts:
- removed P3: buzzer, Pin_Headers:Pin_Header_Straight_1x02, symbol CONN_01X02
- added P16, P17, P18, P3: CONN_01X01, Connect:1pin, symbol CONN_01X01
- added W1, W3, W4: TEST_1P, Pin_Headers:Pin_Header_Straight_1x01, symbol TEST_1P
- C1, C2: value C22uF -> C22pF
- PSU1: symbol DC-DC_Buck -> DC-DC_Buck-RESCUE-extruder
Connections:
- net labels removed: bzr
- wire segments 55 -> 58
- no-connect marks 7 -> 9
